Commit message: edited comments and descriptions.

File: rotors_description/urdf/miniquad.xacro (robot description, xacro)
@@ -1,10 +1,9 @@
 <?xml version="1.0"?>
 <!--
-  Copyright  mrl
+  Copyright 2022, Bilkent University Miniature Robotics Laboratory
 -->
 <robot name="miniquad" xmlns:xacro="http://ros.org/wiki/xacro">
   <!-- Properties (Taken from Novel Dynamic Inversion Architecture Design
 for Quadrocopter Control by Jian Wang et al.)
-NOTE: MINI QUAD ARM LENGTH IS 80 MM * SQRT 2, HERE WE USED 80 SO THA
 -->
   <xacro:property name="namespace" value="$(arg namespace)" />
@@ -12,22 +11,22 @@
   <xacro:property name="use_mesh_file" value="true" />
   <xacro:property name="mesh_file" value="package://rotors_description/meshes/miniquad.dae" />
-  <xacro:property name="mass" value="0.1913" /> <!-- [kg] updated -->
-  <xacro:property name="body_width" value="0.16" /> <!-- [m] updated -->
-  <xacro:property name="body_height" value="0.02" /> <!-- [m] updated -->
-  <xacro:property name="mass_rotor" value="0.00073" /> <!-- [kg] updated-->
-  <xacro:property name="arm_length" value="0.113" /> <!-- [m] updated-->
-  <xacro:property name="rotor_offset_top" value="0.03" /> <!-- [m] updated-->
-  <xacro:property name="radius_rotor" value="0.0445" /> <!-- [m] updated -->
-  <xacro:property name="sin45" value="0.707106781186" />
-  <xacro:property name="cos45" value="0.707106781186" />
-  <xacro:property name="motor_constant" value="7.18e-07" /> <!-- from notespdf -->
-  <xacro:property name="moment_constant" value="0.00944" /> <!-- [m] from notes.pdf, UPDATE: neglecting this caused yaw err. Thus this was recalculated. as 0.00944 -->
-  <xacro:property name="time_constant_up" value="0.0025" /> <!-- [s] default -->
-  <xacro:property name="time_constant_down" value="0.0005" /> <!-- [s] default -->
+  <xacro:property name="mass" value="0.1913" /> <!-- [kg] -->
+  <xacro:property name="body_width" value="0.16" /> <!-- [m] -->
+  <xacro:property name="body_height" value="0.02" /> <!-- [m] -->
+  <xacro:property name="mass_rotor" value="0.00073" /> <!-- [kg] -->
+  <xacro:property name="arm_length" value="0.113" /> <!-- [m] -->
+  <xacro:property name="rotor_offset_top" value="0.03" /> <!-- [m] -->
+  <xacro:property name="radius_rotor" value="0.0445" /> <!-- [m]  -->
+  <xacro:property name="sin45" value="0.707106781186" />  <!-- [rad]  -->
+  <xacro:property name="cos45" value="0.707106781186" />  <!-- [rad]  -->
+  <xacro:property name="motor_constant" value="7.18e-07" /> <!--[Ns/rad] -->
+  <xacro:property name="moment_constant" value="0.00944" /> <!-- [m] -->
+  <xacro:property name="time_constant_up" value="0.0025" /> <!-- [s]  -->
+  <xacro:property name="time_constant_down" value="0.0005" /> <!-- [s]  -->
   <xacro:property name="max_rot_velocity" value="3142" /> <!-- [rad/s] -->
   <xacro:property name="rotor_drag_coefficient" value="0" /> <!-- neglected  -->
-  <xacro:property name="rolling_moment_coefficient" value="0.000000" />  <!-- left as default  -->
+  <xacro:property name="rolling_moment_coefficient" value="0.000000" />  <!-- neglected / set to zero.   -->
   <!-- Property Blocks -->
-  <!-- Body inertia taken from Amirali's matlab code -->
+  <!-- Body inertia is experimentally determined. Taken from Amirali's Simulink simulation.  -->
   <xacro:property name="body_inertia">
     <inertia ixx="0.000399" ixy="0.0" ixz="0.0" iyy="0.000401" iyz="0.0" izz="0.0008" /> <!-- [kg m^2] [kg m^2] [kg m^2] [kg m^2] [kg m^2] [kg m^2] -->

File: rotors_description/urdf/miniquad_base.xacro (robot description, xacro)
@@ -1,18 +1,5 @@
 <?xml version="1.0"?>
 <!--
-  Copyright 2015 Fadri Furrer, ASL, ETH Zurich, Switzerland
-  Copyright 2015 Michael Burri, ASL, ETH Zurich, Switzerland
-  Copyright 2015 Mina Kamel, ASL, ETH Zurich, Switzerland
-  Copyright 2015 Janosch Nikolic, ASL, ETH Zurich, Switzerland
-  Copyright 2015 Markus Achtelik, ASL, ETH Zurich, Switzerland
-  Licensed under the Apache License, Version 2.0 (the "License");
-  you may not use this file except in compliance with the License.
-  You may obtain a copy of the License at
-  http://www.apache.org/licenses/LICENSE-2.0
-  Unless required by applicable law or agreed to in writing, software
-  distributed under the License is distributed on an "AS IS" BASIS,
-  WITHOUT WARRANTIES OR CONDITIONS OF ANY KIND, either express or implied.
-  See the License for the specific language governing permissions and
-  limitations under the License.
+  Copyright 2022, Bilkent University Miniature Robotics Laboratory
 -->
 <robot name="miniquad" xmlns:xacro="http://ros.org/wiki/xacro">

Commit message: temp fix mesh file: replace with hummingbird

File: rotors_description/urdf/miniquad.xacro (robot description, xacro)
@@ -10,5 +10,5 @@
   <xacro:property name="rotor_velocity_slowdown_sim" value="10 " />
   <xacro:property name="use_mesh_file" value="true" />
-  <xacro:property name="mesh_file" value="package://rotors_description/meshes/miniquad.dae" />
+  <xacro:property name="mesh_file" value="package://rotors_description/meshes/hummingbird.dae" />
   <xacro:property name="mass" value="0.1913" /> <!-- [kg] -->
   <xacro:property name="body_width" value="0.16" /> <!-- [m] -->

Commit message: add multi joint model and modify controller
currently crashing, not stable

File: rotors_description/urdf/miniquad.xacro (robot description, xacro)
@@ -7,17 +7,20 @@
 for Quadrocopter Control by Jian Wang et al.)
 -->
-  <xacro:property name="namespace" value="$(arg namespace)" />
+  <xacro:property name="namespace" value="$(arg namespace)"/>
   <xacro:property name="rotor_velocity_slowdown_sim" value="10 " />
-  <xacro:property name="use_mesh_file" value="true" />
+  <xacro:property name="use_mesh_file" value="False" />
   <xacro:property name="mesh_file" value="package://rotors_description/meshes/miniquad.dae" />
   <xacro:property name="mass" value="0.1913" /> <!-- [kg] -->
-  <xacro:property name="body_width" value="0.16" /> <!-- [m] -->
+  <xacro:property name="body_width" value="0.0415" /> <!-- [m] -->
   <xacro:property name="body_height" value="0.02" /> <!-- [m] -->
   <xacro:property name="mass_rotor" value="0.00073" /> <!-- [kg] -->
-  <xacro:property name="arm_length" value="0.113" /> <!-- [m] -->
-  <xacro:property name="rotor_offset_top" value="0.03" /> <!-- [m] -->
+  <xacro:property name="arm_length" value="0.053" /> <!-- [m] -->
+  <xacro:property name="arm_width" value="0.05" /> <!-- [m] -->
+  <xacro:property name="arm_mass" value="0.001" /> <!-- [m] -->
+  <xacro:property name="rotor_offset_top" value="0.005" /> <!-- [m] -->
   <xacro:property name="radius_rotor" value="0.0445" /> <!-- [m]  -->
   <xacro:property name="sin45" value="0.707106781186" />  <!-- [rad]  -->
-  <xacro:property name="cos45" value="0.707106781186" />  <!-- [rad]  -->
+  <xacro:property name="cos45" value="0.707106781186" />
+  <xacro:property name="deg45" value="0.785398163" />  <!-- [rad]  -->
   <xacro:property name="motor_constant" value="7.18e-07" /> <!--[Ns/rad] -->
   <xacro:property name="moment_constant" value="0.00944" /> <!-- [m] -->
@@ -37,15 +40,37 @@
   </xacro:property>
   <!-- Included URDF Files -->
-  <xacro:include filename="$(find rotors_description)/urdf/multirotor_base.xacro" />
+  <xacro:include filename="$(find rotors_description)/urdf/armed_base.xacro" />
   <!-- Instantiate multirotor_base_macro once -->
   <xacro:multirotor_base_macro
+    robot_namespace="${namespace}">
+  </xacro:multirotor_base_macro>
+  <xacro:arm_rotor
     robot_namespace="${namespace}"
-    mass="${mass}"
-    body_width="${body_width}"
-    body_height="${body_height}"
-    use_mesh_file="${use_mesh_file}"
-    mesh_file="${mesh_file}">
-    <xacro:insert_block name="body_inertia" />
-  </xacro:multirotor_base_macro>
+    suffix="back-right"
+    motor_number="0"
+    color="Red">
+    <origin xyz="${body_width*cos45} -${body_width*sin45} 0" rpy="0 0 ${deg45*7}" />
+  </xacro:arm_rotor>
+  <xacro:arm_rotor
+    robot_namespace="${namespace}"
+    suffix="back-left"
+    motor_number="1"
+    color="Red">
+    <origin xyz="${body_width*cos45} ${body_width*sin45} 0" rpy="0 0 ${deg45}" />
+  </xacro:arm_rotor>
+  <xacro:arm_rotor
+    robot_namespace="${namespace}"
+    suffix="front-left"
+    motor_number="2"
+    color="Red">
+    <origin xyz="-${body_width*cos45} ${body_width*sin45} 0" rpy="0 0 ${deg45*3}" />
+  </xacro:arm_rotor>
+  <xacro:arm_rotor
+    robot_namespace="${namespace}"
+    suffix="front-right"
+    motor_number="3"
+    color="Red">
+    <origin xyz="-${body_width*cos45} -${body_width*sin45} 0" rpy="0 0 ${deg45*5}" />
+  </xacro:arm_rotor>
   <!-- Instantiate rotors -->
   <xacro:vertical_rotor
@@ -55,5 +80,5 @@
     motor_constant="${motor_constant}"
     moment_constant="${moment_constant}"
-    parent="${namespace}/base_link"
+    parent="${namespace}/arm_0"
     mass_rotor="${mass_rotor}"
     radius_rotor="${radius_rotor}"
@@ -67,5 +92,5 @@
     use_own_mesh="false"
     mesh="">
-    <origin xyz="${cos45*arm_length} -${sin45*arm_length} ${rotor_offset_top}" rpy="0 0 0" />
+    <origin xyz="${arm_length} 0 ${rotor_offset_top}" rpy="0 0 0" />
     <xacro:insert_block name="rotor_inertia" />
   </xacro:vertical_rotor>
@@ -76,5 +101,5 @@
     motor_constant="${motor_constant}"
     moment_constant="${moment_constant}"
-    parent="${namespace}/base_link"
+    parent="${namespace}/arm_1"
     mass_rotor="${mass_rotor}"
     radius_rotor="${radius_rotor}"
@@ -88,5 +113,5 @@
     use_own_mesh="false"
     mesh="">
-    <origin xyz="${cos45*arm_length} ${sin45*arm_length} ${rotor_offset_top}" rpy="0 0 0" />
+    <origin xyz="${arm_length} 0 ${rotor_offset_top}" rpy="0 0 0" />
     <xacro:insert_block name="rotor_inertia" />
   </xacro:vertical_rotor>
@@ -97,5 +122,5 @@
     motor_constant="${motor_constant}"
     moment_constant="${moment_constant}"
-    parent="${namespace}/base_link"
+    parent="${namespace}/arm_2"
     mass_rotor="${mass_rotor}"
     radius_rotor="${radius_rotor}"
@@ -109,5 +134,5 @@
     use_own_mesh="false"
     mesh="">
-    <origin xyz="-${cos45*arm_length} ${sin45*arm_length} ${rotor_offset_top}" rpy="0 0 0" />
+    <origin xyz="${arm_length} 0 ${rotor_offset_top}" rpy="0 0 0" />
     <xacro:insert_block name="rotor_inertia" />
   </xacro:vertical_rotor>
@@ -118,5 +143,5 @@
     motor_constant="${motor_constant}"
     moment_constant="${moment_constant}"
-    parent="${namespace}/base_link"
+    parent="${namespace}/arm_3"
     mass_rotor="${mass_rotor}"
     radius_rotor="${radius_rotor}"
@@ -130,5 +155,5 @@
     use_own_mesh="false"
     mesh="">
-    <origin xyz="-${cos45*arm_length} -${sin45*arm_length} ${rotor_offset_top}" rpy="0 0 0" />
+    <origin xyz="${arm_length} 0 ${rotor_offset_top}" rpy="0 0 0" />
     <xacro:insert_block name="rotor_inertia" />
   </xacro:vertical_rotor>

File: rotors_description/urdf/miniquad_base.xacro (robot description, xacro)
@@ -3,5 +3,5 @@
   Copyright 2022, Bilkent University Miniature Robotics Laboratory
 -->
-<robot name="miniquad" xmlns:xacro="http://ros.org/wiki/xacro">
+<robot name="mq" xmlns:xacro="http://ros.org/wiki/xacro">
   <xacro:include filename="$(find rotors_description)/urdf/component_snippets.xacro" />
   <!-- Instantiate hummingbird "mechanics" -->
@@ -9,17 +9,16 @@
   <!-- Instantiate a controller. -->
   <xacro:controller_plugin_macro namespace="${namespace}" imu_sub_topic="imu" />
-  <xacro:if value="$(arg enable_mavlink_interface)">
-    <!-- Instantiate mavlink telemetry interface. -->
+  <!-- <xacro:if value="$(arg enable_mavlink_interface)">
     <xacro:default_mavlink_interface namespace="${namespace}" imu_sub_topic="imu" rotor_count="4" />
-  </xacro:if>
+  </xacro:if> -->
   <!-- Mount an ADIS16448 IMU. -->
   <xacro:default_imu namespace="${namespace}" parent_link="${namespace}/base_link" />
   <!-- Mount a GPS. -->
   <xacro:default_gps namespace="${namespace}" parent_link="${namespace}/base_link" />
-  <xacro:if value="$(arg enable_ground_truth)">
+  <!-- <xacro:if value="$(arg enable_ground_truth)">
     <xacro:ground_truth_imu_and_odometry namespace="${namespace}" parent_link="${namespace}/base_link" />
-  </xacro:if>
+  </xacro:if> -->
+<!--
   <xacro:if value="$(arg enable_logging)">
-    <!-- Instantiate a logger -->
     <xacro:bag_plugin_macro
       namespace="${namespace}"
@@ -27,4 +26,4 @@
       rotor_velocity_slowdown_sim="${rotor_velocity_slowdown_sim}"
       wait_to_record_bag="$(arg wait_to_record_bag)" />
-  </xacro:if>
+  </xacro:if> -->
 </robot>
