Commit message: Added multi-joint model for collision

File: rotors_description/urdf/armed_base.xacro (robot description, xacro)
@@ -48,5 +48,5 @@
       <inertial>
         <mass value="0.131" />  <!-- [kg] -->
-        <origin xyz="-0.00694 0.00190 0.02482" />
+        <origin xyz="0.0 0.00 0.0" />  <!-- [m] -->
         <inertia ixx="76498.19e-9" ixy="-138.41e-9" ixz="14011.69e-9" iyy="80911.82e-9" iyz="2914.65e-9" izz="40328.57e-9" />
       </inertial>
@@ -77,6 +77,6 @@
     params="robot_namespace suffix motor_number *origin color">
     <joint name="${robot_namespace}/arm_${motor_number}_joint" type="revolute" >
-      <limit lower="-1.52" upper="1.52" effort="-1" velocity="-1"/>
-      <dynamics damping="1" friction="1" />
+      <limit lower="-2" upper="2" effort="100" velocity="100"/>
+      <dynamics damping="0.0001" friction="0.0001" />
       <xacro:insert_block name="origin" />
       <axis xyz="0 0 1" />
@@ -137,5 +137,5 @@
         <mass value="0.0071" /> <!-- [kg] -->
         <origin xyz="23.51e-3 0 -3.48e-3" rpy="0 0 0" />
-        <inertia ixx="302.58e-9" ixy="0" ixz="55.52" iyy="569.34e-9" iyz="0" izz="841.34e-9" />
+        <inertia ixx="302.58e-9" ixy="0" ixz="55.52e-9" iyy="569.34e-9" iyz="0" izz="841.34e-9" />
       </inertial>
       <visual>
@@ -155,4 +155,12 @@
       <material>Gazebo/${color}</material>
     </gazebo>
+    <gazebo>
+    <!-- joint torsional spring plugin -->
+    <plugin name="arm_${motor_number}_joint_torsional_spring" filename="libgazebo_joint_torsional_spring.so">
+      <kx>0.5</kx>
+      <set_point>0.0</set_point>
+      <joint>${robot_namespace}/arm_${motor_number}_joint</joint>
+    </plugin>
+  </gazebo>
   </xacro:macro>
   <!-- Rotor joint and link -->

File: rotors_description/urdf/miniquad.xacro (robot description, xacro)
@@ -18,4 +18,5 @@
   <xacro:property name="arm_width" value="0.05" /> <!-- [m] -->
   <xacro:property name="arm_mass" value="0.001" /> <!-- [m] -->
+  <xacro:property name="rotor_dist" value="0.053" /> <!-- [m] -->
   <xacro:property name="rotor_offset_top" value="0.005" /> <!-- [m] -->
   <xacro:property name="radius_rotor" value="0.0445" /> <!-- [m]  -->
@@ -76,5 +77,5 @@
   <xacro:vertical_rotor
     robot_namespace="${namespace}"
-    suffix="front-right"
+    suffix="back-right"
     direction="cw"
     motor_constant="${motor_constant}"
@@ -97,5 +98,5 @@
   <xacro:vertical_rotor
     robot_namespace="${namespace}"
-    suffix="back-right"
+    suffix="back-left"
     direction="ccw"
     motor_constant="${motor_constant}"
@@ -118,5 +119,5 @@
   <xacro:vertical_rotor
     robot_namespace="${namespace}"
-    suffix="back-left"
+    suffix="front-left"
     direction="cw"
     motor_constant="${motor_constant}"
@@ -139,5 +140,5 @@
   <xacro:vertical_rotor
     robot_namespace="${namespace}"
-    suffix="front-left"
+    suffix="front-right"
     direction="ccw"
     motor_constant="${motor_constant}"
